File: 03 - Hardware/05-Prototype-UpdatedComponents/05-Prototype-UpdatedComponents.kicad_pcb (KiCad board)
At the start: 2 copper layers, 15 parts, among them J1 4P4C, J2 4P4C, U1 YAAJ_BluePill, U3 BME280_I2C_New_LK888, U4 SX1278_Minimal, U5 microSD_Module_3V3_Horizontal, U6 MCP6002-xP

Commit message: Schematic update
Parts:
- added C0: 220n, Custom_Libs:C_Radial_W5.5mm_H9.0mm_T3.0mm_P4.3mm, F.Cu at (88.4, 100.3)
- added C5: 220n, Custom_Libs:C_Radial_W5.5mm_H9.0mm_T3.0mm_P4.3mm, F.Cu at (88.4, 96.1)
- added J0: Conn_01x03_Male, Connector_PinSocket_2.54mm:PinSocket_1x03_P2.54mm_Vertical, F.Cu at (81.9, 108.8)
- added J3: Conn_01x03_Male, Connector_PinSocket_2.54mm:PinSocket_1x03_P2.54mm_Vertical, F.Cu at (54.1, 29.2)
- added R1: 3.3k, Resistor_THT:R_Axial_DIN0204_L3.6mm_D1.6mm_P5.08mm_Horizontal, F.Cu at (78.3, 95.5)
- added R4: 3.3k, Resistor_THT:R_Axial_DIN0204_L3.6mm_D1.6mm_P5.08mm_Horizontal, F.Cu at (78.3, 98.7)
- added U2: DS3231_Module_FullAccess, DS3231_Module:DS3231_Module_FullSize, F.Cu at (46.0, 109.1)
- moved U0 83.7 mm to (135.4, 97.9), turned to 90 degrees
- renumbered R1 to R0, R4 to R5, U1 to U0, U5 to U1, U4 to U3, U6 to U4, U3 to U5
Connections:
- net Net-(C1-Pad1) renamed /Passive LPF
- J1 pad 1: unconnected-(J1-Pad1) -> GND
- J1 pad 2: unconnected-(J1-Pad2) -> GND
- J1 pad 3: unconnected-(J1-Pad3) -> Anemometer
- J2 pad 2: unconnected-(J2-Pad2) -> GND
- J2 pad 3: unconnected-(J2-Pad3) -> Rain gauge
- U0 pad 1: unconnected-(U1-Pad1) -> LoRa_NCSS
- U0 pad 2: unconnected-(U1-Pad2) -> LoRa_SCLK
- U0 pad 26: unconnected-(U1-Pad26) -> Rain gauge
- U0 pad 28: unconnected-(U1-Pad28) -> Anemometer
- U0 pad 3: unconnected-(U1-Pad3) -> LoRa_MISO
- U0 pad 4: unconnected-(U1-Pad4) -> LoRa_MOSI
- U0 pad 5: unconnected-(U1-Pad5) -> LoRa_Reset
- U0 pad 8: unconnected-(U1-Pad8) -> LoRa_DIO0
- U3 pad 1: unconnected-(U4-Pad1) -> GND
- U3 pad 2: unconnected-(U4-Pad2) -> +3.3VP
- U3 pad 3: unconnected-(U4-Pad3) -> LoRa_Reset
- U3 pad 4: unconnected-(U4-Pad4) -> LoRa_NCSS
- U3 pad 5: unconnected-(U4-Pad5) (its old number) -> LoRa_SCLK
- U3 pad 6: unconnected-(U4-Pad6) (its old number) -> LoRa_MOSI
- U3 pad 7: unconnected-(U4-Pad7) (its old number) -> LoRa_MISO
- U3 pad 8: unconnected-(U4-Pad8) -> LoRa_DIO0

Commit message: Update PCB
Parts:
- added C0: 1u, Capacitor_THT:CP_Radial_D5.0mm_P2.00mm, F.Cu at (104.1, 58.4)
- added C1: 1u, Capacitor_THT:CP_Radial_D5.0mm_P2.00mm, F.Cu at (110.8, 58.4)
- added J0: Barrel_Jack, Connector_BarrelJack:BarrelJack_Horizontal, F.Cu at (84.7, 28.8)
- added R0: 240, Resistor_THT:R_Axial_DIN0204_L3.6mm_D1.6mm_P5.08mm_Horizontal, F.Cu at (88.7, 31.0)
- added R1: 390, Resistor_THT:R_Axial_DIN0204_L3.6mm_D1.6mm_P5.08mm_Horizontal, F.Cu at (83.2, 40.8)
- added R2: 240, Resistor_THT:R_Axial_DIN0204_L3.6mm_D1.6mm_P5.08mm_Horizontal, F.Cu at (83.2, 37.7)
- added R3: 390, Resistor_THT:R_Axial_DIN0204_L3.6mm_D1.6mm_P5.08mm_Horizontal, F.Cu at (88.7, 34.2)
- added U1: LM317_TO-220, Package_TO_SOT_THT:TO-220-3_Vertical, F.Cu at (73.4, 40.0)
- added U2: LM317_TO-220, Package_TO_SOT_THT:TO-220-3_Vertical, F.Cu at (90.5, 27.4)
- moved U3 196.4 mm to (254.0, 124.5), turned to 180 degrees
- moved J2 153.6 mm to (180.3, 142.2)
- moved U5 150.2 mm to (198.1, 45.7), turned to -90 degrees
- moved U6 141.8 mm to (216.5, 125.1), turned to -90 degrees
- moved J3 123.4 mm to (162.6, 142.2)
- moved R7 122.3 mm to (208.9, 121.9)
- moved C5 110.4 mm to (196.2, 127.0), turned to -90 degrees
- moved R5 109.0 mm to (180.3, 134.0), turned to 180 degrees
- moved C6 107.8 mm to (201.9, 127.0), turned to -90 degrees
- moved C4 103.9 mm to (190.5, 127.0), turned to -90 degrees
- moved R4 101.2 mm to (180.3, 129.5), turned to 180 degrees
- moved R6 99.7 mm to (175.3, 125.1)
- moved C3 94.7 mm to (184.8, 127.0), turned to -90 degrees
- moved C2 88.2 mm to (170.2, 133.3)
- moved U0 70.7 mm to (204.5, 82.7), turned to -90 degrees
- renumbered C0 to C2, C1 to C3, C2 to C4, C3 to C5, C4 to C6, C5 to C7, J0 to J1, J1 to J2, J2 to J3, J3 to J4, R0 to R4, R1 to R5, R2 to R6, R3 to R7, R4 to R8, R5 to R9, U1 to U3, U2 to U4, U3 to U5, U4 to U6, U5 to U7
Connections:
- U0 pad 6: unconnected-(U0-Pad6) -> UART_TX
- U0 pad 7: unconnected-(U0-Pad7) -> UART_RX

Commit message: Update PCB
Parts:
- moved U3 108.1 mm to (146.1, 130.8), turned to 90 degrees
- moved R8 92.9 mm to (165.7, 130.2), turned to 180 degrees
- moved C7 83.0 mm to (166.4, 124.5), turned to 90 degrees
- moved U7 82.1 mm to (160.0, 91.4)
- moved U5 29.6 mm to (205.7, 74.3)
- moved U0 19.1 mm to (201.9, 101.6)
- moved R7 16.0 mm to (193.0, 123.8), turned to 180 degrees
- moved U6 9.61 mm to (207.0, 123.8), turned to 0 degrees
- moved C2 8.98 mm to (171.4, 124.5), turned to 90 degrees
- moved C3 1.27 mm to (184.8, 128.3)
- moved C4 1.27 mm to (190.5, 128.3)
- moved C5 1.27 mm to (196.2, 128.3)
- moved C6 1.27 mm to (201.9, 128.3)
- moved R5 0.64 mm to (180.3, 133.3)
- moved R6 0.64 mm to (175.3, 125.7)
Routing:
- net GND: track 0.00 -> 191.9 mm
- net +3V3: track 0.00 -> 167.1 mm, vias 0 -> 1
- net SPI1_SCK: track 0.00 -> 81.0 mm, vias 0 -> 1
- net SPI1_MOSI: track 0.00 -> 55.7 mm
- net MICROSD_NCSS: track 0.00 -> 55.3 mm
- net SPI1_MISO: track 0.00 -> 44.5 mm
- net WindVane_filtered: track 0.00 -> 31.2 mm
- net Rain gauge: track 0.00 -> 30.8 mm
- net Anemometer: track 0.00 -> 28.9 mm
- net /Passive LPF: track 0.00 -> 28.0 mm
- net WindVane_raw: track 0.00 -> 20.9 mm
- net I2C_CLK: track 0.00 -> 18.7 mm
- net I2C_SDA: track 0.00 -> 9.22 mm

Commit message: First version of updated board
Parts:
- added J2: Conn_01x03_Male, Connector_PinSocket_2.54mm:PinSocket_1x03_P2.54mm_Vertical, B.Cu at (143.8, 118.3)
- C1, J1, R0, R1, R2, R3, R9, U4: moved to B.Cu
- moved U1 156.1 mm to (212.4, 111.1), turned to -90 degrees
- moved R0 151.7 mm to (215.9, 113.7), turned to 90 degrees
- moved R2 147.6 mm to (215.9, 102.2), turned to 90 degrees
- moved R1 145.9 mm to (212.7, 108.0), turned to 180 degrees
- moved U2 141.8 mm to (212.4, 99.7), turned to -90 degrees
- moved J0 140.1 mm to (210.5, 90.5), turned to 180 degrees
- moved R3 135.8 mm to (207.6, 99.7), turned to -90 degrees
- moved J5 134.9 mm to (171.4, 95.9), turned to 180 degrees
- moved R9 118.5 mm to (163.8, 104.8)
- moved C0 117.2 mm to (207.6, 113.4), turned to 90 degrees
- moved U4 115.9 mm to (160.7, 92.1), turned to 180 degrees
- moved C1 82.0 mm to (184.8, 93.7), turned to -90 degrees
- moved J1 61.7 mm to (143.5, 105.4), turned to -90 degrees
- moved U5 17.1 mm to (193.0, 85.7)
- moved R5 13.9 mm to (167.0, 129.5), turned to 0 degrees
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- renumbered J2 to J3, J3 to J4, J4 to J5
Routing:
- net GND: track 191.9 -> 332.8 mm
- net +3V3: track 167.1 -> 245.5 mm, vias 1 -> 0
- net RTC_ALARM: track 0.00 -> 69.6 mm
- net LoRa_SCLK: track 0.00 -> 63.8 mm
- net UART_TX: track 0.00 -> 53.9 mm
- net UART_RX: track 0.00 -> 49.4 mm
- net I2C_SDA: track 9.22 -> 56.7 mm
- net +VDC: track 0.00 -> 43.1 mm
- net +3.3VP: track 0.00 -> 42.6 mm
- net LoRa_MOSI: track 0.00 -> 34.2 mm
- net I2C_CLK: track 18.7 -> 43.1 mm
- net LoRa_DIO0: track 0.00 -> 24.2 mm
- net /32768Hz out: track 0.00 -> 21.7 mm
- net DS18B20: track 0.00 -> 21.2 mm
- net LoRa_NCSS: track 0.00 -> 20.9 mm
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- added copper zone on B.Cu, net GND
- added copper zone on F.Cu, net GND
Other:
- board outline added: 83.7 x 70.6 mm
