File: 03 - Hardware/05-Prototype-UpdatedComponents/05-Prototype-UpdatedComponents.kicad_sch (KiCad schematic)
At the start: 8 parts

Commit message: hardware update
Parts:
- removed J?: Screw_Terminal_01x03, symbol Connector:Screw_Terminal_01x03
- added C1: 10n, Custom_Libs:C_Radial_W5.5mm_H9.0mm_T3.0mm_P4.3mm, symbol Device:C
- added C2: 4.7n, Custom_Libs:C_Radial_W5.5mm_H9.0mm_T3.0mm_P4.3mm, symbol Device:C
- added C3: 3.3n, Custom_Libs:C_Radial_W5.5mm_H9.0mm_T3.0mm_P4.3mm, symbol Device:C
- added C4: 2.2n, Custom_Libs:C_Radial_W5.5mm_H9.0mm_T3.0mm_P4.3mm, symbol Device:C
- added J3: Conn_01x03_Male, symbol Connector:Conn_01x03_Male
- added R1, R3: 3.3k, Resistor_THT:R_Axial_DIN0204_L3.6mm_D1.6mm_P5.08mm_Horizontal, symbol Device:R
- added R2: 680, Resistor_THT:R_Axial_DIN0204_L3.6mm_D1.6mm_P5.08mm_Horizontal, symbol Device:R
- added R4: 4.7k, Resistor_THT:R_Axial_DIN0204_L3.6mm_D1.6mm_P5.08mm_Horizontal, symbol Device:R
- added U6: MCP6002-xP, Package_DIP:DIP-8_W7.62mm_LongPads, symbol Amplifier_Operational:MCP6002-xP
- U1: renamed from U?; footprint (none) -> KiCAD_STM32_BluePill:YAAJ_BluePill_1
- U3: renamed from U?; footprint BME280_Module:BME280_I2C -> BME280_Module:BME280_I2C_Small
- U5: renamed from U?; value (none) -> microSD_Module_3V3_Horizontal; footprint (none) -> Custom_Libs:microSD_mini
- gave numbers to parts that had none: 4
Connections:
- net GND: now also U2.4 (GND), U3.2 (GND), U3.5 (ADDR), U4.1 (GND), U5.6 (GND), C1.2, C2.2, C3.2, C4.2, J3.1 (Pin_1), R3.1, U6.4 (V-)
- net WindVane_raw: now reaches J1.4
- net WindVane_raw: now also R1.2, R2.1
- net +3V3: now reaches U3.1 (VCC)
- net +3V3: now also U1.20 (3V3), U1.38 (3V3), U2.3 (VCC), U5.1 (3V3), J3.3 (Pin_3), R1.1, R4.1, U6.8 (V+)
- net I2C_CLK: now reaches U3.3 (SCL)
- net I2C_CLK: now also U1.14 (PB6), U2.1 (SCL)
- net I2C_SDA: now reaches U3.4 (SDA)
- net I2C_SDA: now also U1.15 (PB7), U2.2 (SDA)
- net LoRa_NCSS: now reaches U1.1 (PB12)
- net LoRa_NCSS: now also U4.4 (NCSS)
- net RTC_ALARM: now reaches U1.10 (PA15)
- net RTC_ALARM: now also U2.6 (SQW)
- net DS18B20: now reaches U1.11 (PB3)
- net DS18B20: now also J3.2 (Pin_2), R4.2
- net LoRa_SCLK: now reaches U1.2 (PB13)
- net LoRa_SCLK: now also U4.5 (SCLK)
- net MICROSD_NCSS: now reaches U1.29 (PA4)
- net MICROSD_NCSS: now also U5.2 (CS)
- net LoRa_MISO: now reaches U1.3 (PB14)
- net LoRa_MISO: now also U4.7 (MISO)
- net SPI1_SCK: now reaches U1.30 (PA5)
- net SPI1_SCK: now also U5.4 (CLK)
- net SPI1_MISO: now reaches U1.31 (PA6)
- net SPI1_MISO: now also U5.5 (MISO)
- net SPI1_MOSI: now reaches U1.32 (PA7)
- net SPI1_MOSI: now also U5.3 (MOSI)
- net WindVane_filtered: now reaches U1.34 (PB1)
- net WindVane_filtered: now also R3.2, U6.1, U6.2 (-)
- net LoRa_MOSI: now reaches U1.4 (PB15)
- net LoRa_MOSI: now also U4.6 (MOSI)
- net LoRa_Reset: now reaches U1.5 (PA8)
- net LoRa_Reset: now also U4.3 (RST)
- net LoRa_DIO0: now reaches U1.8 (PA11)
- net LoRa_DIO0: now also U4.8 (DIO0)
- net +3.3VP: now reaches U4.2 (VCC)
- new net: C1.1, C2.1, C3.1, C4.1, R2.2, U6.3 (+)
- no-connect marks 2 -> 19
Other:
- note added: "RJ11 connector for anemometer and windvane"
- note added: "RJ11 connector for rain gauge"
- moved on the sheet: J2, U3, U5

Commit message: Schematic update
Parts:
- added C0, C5: 220n, Custom_Libs:C_Radial_W5.5mm_H9.0mm_T3.0mm_P4.3mm, symbol Device:C
- added J0: Conn_01x03_Male, Connector_PinSocket_2.54mm:PinSocket_1x03_P2.54mm_Vertical, symbol Connector:Conn_01x03_Male
- added R1, R4: 3.3k, Resistor_THT:R_Axial_DIN0204_L3.6mm_D1.6mm_P5.08mm_Horizontal, symbol Device:R
- J3: footprint (none) -> Connector_PinSocket_2.54mm:PinSocket_1x03_P2.54mm_Vertical
- U2: footprint (none) -> DS3231_Module:DS3231_Module_FullSize
- renumbered R1 to R0, R4 to R5, U1 to U0, U5 to U1, U4 to U3, U6 to U4, U3 to U5
Connections:
- net +3V3: now also R1.1, R4.1
- net GND: now also J1.1, J1.2, J2.2, C0.1, C5.1, J0.1 (Pin_1), J0.3 (Pin_3)
- net Anemometer: now reaches J1.3
- net Anemometer: now also U0.28 (PA3), C0.2, R1.2
- net Rain gauge: now reaches U0.26 (PA1)
- net Rain gauge: now also J2.3, C5.2, R4.2
- net UART_TX: now reaches U0.6 (PA9)
- net UART_RX: now reaches U0.7 (PA10)
- net Passive LPF: now reaches C1.1, C2.1, C3.1, C4.1, R2.2, U4.3 (+)
- net 32768Hz out: now reaches U2.5 (32K)
- net 32768Hz out: now also J0.2 (Pin_2)
- no-connect marks 19 -> 21
Other:
- note added: "32768-Hz output for manual calibration"
- note added: "Analogue filter for wind vane input"
- note added: "BME280: - Temperature - Humidity - Barometric Pressure"
- note added: "Connector for DS18B20 sensor: - Temperature"
- note added: "Local data storage: microSD"
- note added: "Microcontroller unit: STM32F103CBT6 on Blue Pill"
- note added: "RJ11 connector for anemometer (wind speed) and wind vane (wind direction)"
- note added: "Sensor units"
- note added: "Time keeper unit: DS3231 RTC"
- note added: "Wireless communication unit: LoRa by SX1278"
- note removed: "RJ11 connector for anemometer and windvane"
- moved on the sheet: C1, C2, C3, C4, J1, J2, J3, R0, R2, R3, R5, U0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

Commit message: Update PCB
Parts:
- added C0, C1: (no value), symbol Device:C_Polarized_Small
- added J0: (no value), symbol Connector:Barrel_Jack_Switch
- added R0, R1, R2, R3: (no value), symbol Device:R
- added U1, U2: (no value), symbol Regulator_Linear:LM317_TO-220
- C2: renamed from C0; value 220n -> (none); footprint Custom_Libs:C_Radial_W5.5mm_H9.0mm_T3.0mm_P4.3mm -> (none)
- C3: renamed from C1; value 10n -> (none); footprint Custom_Libs:C_Radial_W5.5mm_H9.0mm_T3.0mm_P4.3mm -> (none)
- C4: renamed from C2; value 4.7n -> (none); footprint Custom_Libs:C_Radial_W5.5mm_H9.0mm_T3.0mm_P4.3mm -> (none)
- C5: renamed from C3; value 3.3n -> (none); footprint Custom_Libs:C_Radial_W5.5mm_H9.0mm_T3.0mm_P4.3mm -> (none)
- C6: renamed from C4; value 2.2n -> (none); footprint Custom_Libs:C_Radial_W5.5mm_H9.0mm_T3.0mm_P4.3mm -> (none)
- C7: renamed from C5; value 220n -> (none); footprint Custom_Libs:C_Radial_W5.5mm_H9.0mm_T3.0mm_P4.3mm -> (none)
- J1: renamed from J0; value Conn_01x03_Male -> (none); footprint Connector_PinSocket_2.54mm:PinSocket_1x03_P2.54mm_Vertical -> (none)
- J2: renamed from J1; value 4P4C -> (none); footprint RJ11-Connectors:4P4C -> (none)
- J3: renamed from J2; value 4P4C -> (none); footprint RJ11-Connectors:4P4C -> (none)
- J4: renamed from J3; value Conn_01x03_Male -> (none); footprint Connector_PinSocket_2.54mm:PinSocket_1x03_P2.54mm_Vertical -> (none)
- R4: renamed from R0; value 3.3k -> (none); footprint Resistor_THT:R_Axial_DIN0204_L3.6mm_D1.6mm_P5.08mm_Horizontal -> (none)
- R5: renamed from R1; value 3.3k -> (none); footprint Resistor_THT:R_Axial_DIN0204_L3.6mm_D1.6mm_P5.08mm_Horizontal -> (none)
- R6: renamed from R2; value 680 -> (none); footprint Resistor_THT:R_Axial_DIN0204_L3.6mm_D1.6mm_P5.08mm_Horizontal -> (none)
- R7: renamed from R3; value 3.3k -> (none); footprint Resistor_THT:R_Axial_DIN0204_L3.6mm_D1.6mm_P5.08mm_Horizontal -> (none)
- R8: renamed from R4; value 3.3k -> (none); footprint Resistor_THT:R_Axial_DIN0204_L3.6mm_D1.6mm_P5.08mm_Horizontal -> (none)
- R9: renamed from R5; value 4.7k -> (none); footprint Resistor_THT:R_Axial_DIN0204_L3.6mm_D1.6mm_P5.08mm_Horizontal -> (none)
- U3: renamed from U1; value microSD_Module_3V3_Horizontal -> (none); footprint Custom_Libs:microSD_mini -> (none)
- U4: renamed from U2; value DS3231_Module_FullAccess -> (none); footprint DS3231_Module:DS3231_Module_FullSize -> (none)
- U5: renamed from U3; value SX1278_Minimal -> (none); footprint SX1278_Module:SX1278_Minimal -> (none)
- U6: renamed from U4; value MCP6002-xP -> (none); footprint Package_DIP:DIP-8_W7.62mm_LongPads -> (none)
- U7: renamed from U5; value BME280_I2C_New_LK888 -> (none); footprint BME280_Module:BME280_I2C_Small -> (none)
- renumbered U4 to U6
Connections:
- net +3.3VP: now also C1.1, R2.1, U2.2 (VO)
- net +3V3: now also C0.1, R0.1, U1.2 (VO)
- net GND: now also C0.2, C1.2, J0.2, J0.3, R1.2, R3.2
- new net +VDC: J0.1, U1.3 (VI), U2.3 (VI)
- new net V_adj: R0.2, R1.1, U1.1 (ADJ)
- new net V_adj_VP: R2.2, R3.1, U2.1 (ADJ)
Other:
- note added: "External power supply for PCB"
- note added: "Regulated +3.3V supply"
- note added: "Separate +3.3VP for SX1278"
- moved on the sheet: C2, C3, C4, C5, C6, C7, J1, J2, J3, J4, R4, R5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

Commit message: First version of updated board
Parts:
- added J2: (no value), symbol Connector:Conn_01x03_Male
- C0, C1: value (none) -> 1u; footprint (none) -> Capacitor_THT:CP_Radial_D5.0mm_P2.00mm
- C2, C7: value (none) -> 220n; footprint (none) -> Custom_Libs:C_Radial_W5.5mm_H9.0mm_T3.0mm_P4.3mm
- C3: value (none) -> 10n; footprint (none) -> Custom_Libs:C_Radial_W5.5mm_H9.0mm_T3.0mm_P4.3mm
- C4: value (none) -> 4.7n; footprint (none) -> Custom_Libs:C_Radial_W5.5mm_H9.0mm_T3.0mm_P4.3mm
- C5: value (none) -> 3.3n; footprint (none) -> Custom_Libs:C_Radial_W5.5mm_H9.0mm_T3.0mm_P4.3mm
- C6: value (none) -> 2.2n; footprint (none) -> Custom_Libs:C_Radial_W5.5mm_H9.0mm_T3.0mm_P4.3mm
- J0: value (none) -> Barrel_Jack; footprint (none) -> Connector_BarrelJack:BarrelJack_Horizontal
- J1: value (none) -> Conn_01x03_Male; footprint (none) -> Connector_PinSocket_2.54mm:PinSocket_1x03_P2.54mm_Vertical
- R0, R2: value (none) -> 240; footprint (none) -> Resistor_THT:R_Axial_DIN0204_L3.6mm_D1.6mm_P5.08mm_Horizontal
- R1, R3: value (none) -> 390; footprint (none) -> Resistor_THT:R_Axial_DIN0204_L3.6mm_D1.6mm_P5.08mm_Horizontal
- R4, R5, R7, R8: value (none) -> 3.3k; footprint (none) -> Resistor_THT:R_Axial_DIN0204_L3.6mm_D1.6mm_P5.08mm_Horizontal
- R6: value (none) -> 680; footprint (none) -> Resistor_THT:R_Axial_DIN0204_L3.6mm_D1.6mm_P5.08mm_Horizontal
- R9: value (none) -> 4.7k; footprint (none) -> Resistor_THT:R_Axial_DIN0204_L3.6mm_D1.6mm_P5.08mm_Horizontal
- U1, U2: value (none) -> LM317_TO-220; footprint (none) -> Package_TO_SOT_THT:TO-220-3_Vertical
- U3: value (none) -> microSD_Module_3V3_Horizontal; footprint (none) -> Custom_Libs:microSD_mini
- U5: value (none) -> SX1278_Minimal; footprint (none) -> SX1278_Module:SX1278_Minimal
- U6: value (none) -> MCP6002-xP; footprint (none) -> Package_DIP:DIP-8_W7.62mm_LongPads
- U7: value (none) -> BME280_I2C_New_LK888; footprint (none) -> BME280_Module:BME280_I2C_Small
- renumbered J2 to J3, J3 to J4, J4 to J5
Connections:
- net GND: now also J2.1 (Pin_1)
- net UART_RX: now also J2.3 (Pin_3)
- net UART_TX: now also J2.2 (Pin_2)
Other:
- note added: "Communication units"
- note added: "LoRa with SX1278"
- note added: "UART"
- note removed: "Wireless communication unit: LoRa by SX1278"
- moved on the sheet: U5

Commit message: 4
Parts:
- added BT1, BT2: (no value), symbol Device:Battery_Cell
- added Q? (x2): (no value), symbol Device:Q_PMOS_GDS
- added Q?: P MOSFET, symbol Device:Q_PMOS_GDS
- added R_{1}, R_{1}? (x2), R_{2}: (no value), symbol Device:R
- added R_{1}? (x2): 240, Resistor_THT:R_Axial_DIN0204_L3.6mm_D1.6mm_P5.08mm_Horizontal, symbol Device:R
- added R_{2}? (x2): 390, Resistor_THT:R_Axial_DIN0204_L3.6mm_D1.6mm_P5.08mm_Horizontal, symbol Device:R
- added SC?: (no value), symbol Device:Solar_Cells
- added U: (no value), symbol Amplifier_Operational:MCP6002-xP
- added U?: (no value), Package_TO_SOT_THT:TO-220-3_Vertical, symbol Regulator_Linear:LM317_TO-220
- added U? (x2): LM317, Package_TO_SOT_THT:TO-220-3_Vertical, symbol Regulator_Linear:LM317_TO-220
- C2, C7: value 220n -> 68n
- J2, J5: value (none) -> Conn_01x03_Male; footprint (none) -> Connector_PinSocket_2.54mm:PinSocket_1x03_P2.54mm_Vertical
- J3, J4: value (none) -> 4P4C; footprint (none) -> RJ11-Connectors:4P4C
- R4: value 3.3k -> 3k
- R5, R8: value 3.3k -> 33k
- U4: value (none) -> DS3231_Module_FullAccess; footprint (none) -> DS3231_Module:DS3231_Module_FullSize
Connections:
- net +3.3VP: no longer U5.2 (VCC)
- net +3V3: now also U5.2 (VCC), Q?.2 (D), Q?.2 (D), U.3 (+), U.5 (+), U.8 (V+)
- net GND: now also R_{2}.2, R_{2}?.2, R_{2}?.2, SC?.2 (-), U.4 (V-)
- net Rain gauge: no longer U0.26 (PA1)
- net WindVane_filtered renamed Wind_Vane
- new net: SC?.1 (+), U?.3 (VI)
- new net: Q?.1 (G), R_{1}?.2 (x2)
- new net: Q?.3 (S), R_{1}?.1, U.6 (-), U?.2 (VO)
- new net: Q?.3 (S), R_{1}.1, U.2 (-), U?.2 (VO)
- new net: R_{1}.2, R_{2}.1, U?.1 (ADJ)
- new net: R_{1}?.1, U.1
- new net: Q?.3 (S), R_{1}?.1, U?.2 (VO)
- new net: R_{1}?.2, R_{2}?.1, U?.1 (ADJ) (x2)
- new net: BT1.2 (-), BT2.1 (+)
- new net: R_{1}?.1, U.7
- new net Rain_Gauge: U0.26 (PA1)
- new net VD: Q?.2 (D), U?.3 (VI)
Other:
- note added: "3.3V regulator"
- note added: "B+"
- note added: "B-"
- note added: "BM"
- note added: "HX-2S-D20 battery charger"
- note added: "Main station"
- note added: "P+"
- note added: "P-"
- note added: "Reverse current protection circuit"
- note added: "V_{in}"
- note added: "V_{out}"
- note added: "Vin+"
- note added: "Vin-"
- note added: "Vout+"
- note added: "Vout-"
- note added: "XL4015 Buck Converter"
