File: 01 - Simulations/Archive - from Senior Project/LPF/Analog RC Filter/RC-LPF/RC-LPF.kicad_sch (KiCad schematic)
At the start: 7 parts

Commit message: 4
Parts:
- added C4: 2.2n, symbol Device:C
- added C?: 68n, symbol Device:C
- added R_pullup30: 33k, symbol Device:R
- added R_{pulldown}: (no value), symbol Device:R
- added R_{pullup}: 4.7k, symbol Device:R
- added SW?: SW_Reed, symbol Switch:SW_Reed
- added U0, U? (x2): MCP6002-xMC, Package_DFN_QFN:DFN-8-1EP_3x2mm_P0.5mm_EP1.75x1.45mm, symbol Amplifier_Operational:MCP6002-xMC
- added U?: DS18B20, Package_TO_SOT_THT:TO-92_Inline, symbol Sensor_Temperature:DS18B20
- C1: renamed from C0; value (none) -> 10n
- C2: renamed from C1; value (none) -> 4.7n
- C3: renamed from C2; value (none) -> 3.3n
- R?: value (none) -> R_{WindVane}
- R_{filter}: renamed from R_filter; value (none) -> 680
- R_{pullup}: renamed from R_pullup; value (none) -> 3k
- SW?: value (none) -> SW_Reed
Connections:
- net +3V3: now also R_pullup30.1, R_{pullup}.1, U0.8 (V+), U?.3 (VDD)
- net GND: now also C4.2, C?.2, R_{pulldown}.1, SW?.1, U0.4 (V-), U0.9 (V-), U?.1 (GND)
- net at C1.1, C2.1, C3.1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: now also C4.1, U?.3 (+)
- new net Anemometer: C?.1, R_pullup30.2, SW?.2
- new net DS18B20: R_{pullup}.2
- new net Wind_Vane: R_{pulldown}.2, U?.1, U?.2 (-)
- no-connect marks 0 -> 3
Other:
- note added: "Anemometer"
- note added: "One-Wire Bus"
- note removed: "ADC module"
